Commit message: stl, dae file directory replaced

File: end_effectors/common/utils.xacro (robot description, xacro)
@@ -37,10 +37,10 @@
       <visual name="${prefix}${name}_visual">
         <geometry>
-          <mesh filename="package://${description_pkg}/meshes/robot_ee/${ee_id}/visual/${name}.dae" />
+          <mesh filename="file://$(find franka_description)/meshes/robot_ee/${ee_id}/visual/${name}.dae" />
         </geometry>
       </visual>
       <collision name="${prefix}${name}_collision">
         <geometry>
-          <mesh filename="package://franka_description/meshes/robot_ee/${ee_id}/collision/${name}.stl" />
+          <mesh filename="file://$(find franka_description)/meshes/robot_ee/${ee_id}/collision/${name}.stl" />
         </geometry>
       </collision>

File: robots/common/utils.xacro (robot description, xacro)
@@ -38,10 +38,10 @@
       <visual name="${prefix}${name}_visual">
         <geometry>
-          <mesh filename="package://${description_pkg}/meshes/robot_arms/${arm_id}/visual/${name}.dae" />
+          <mesh filename="file://$(find franka_description)/meshes/robot_arms/${arm_id}/visual/${name}.dae" />
         </geometry>
       </visual>
       <collision name="${prefix}${name}_collision">
         <geometry>
-          <mesh filename="package://franka_description/meshes/robot_arms/${arm_id}/collision/${name}.stl" />
+          <mesh filename="file://$(find franka_description)/meshes/robot_arms/${arm_id}/collision/${name}.stl" />
         </geometry>
       </collision>
