Commit message: camera shape done

File: robots/common/franka_robot.xacro (robot description, xacro)
@@ -69,5 +69,29 @@
       />
     </xacro:if>
-    <xacro:if value="${hand and ee_id != 'none' and ee_id != 'franka_hand'}">
+    <xacro:if value="${hand and ee_id == 'camera'}">
+      <!-- camera.xacro 포함 -->
+      <xacro:include filename="$(find franka_description)/end_effectors/common/camera.xacro" />
+      <xacro:include filename="$(find franka_description)/end_effectors/$(arg ee_id)/$(arg ee_id)_arguments.xacro" />
+      <xacro:property name="special_connection" value="$(arg special_connection)" />
+      <xacro:property name="connection" value="${special_connection if special_connection != '' else arm_id + '_link8'}" />
+      <!-- <xacro:property name="connection" value="arm_id + '_link8'" /> -->
+      <!-- camera 매크로 호출 -->
+      <xacro:camera
+        connected_to="${arm_prefix_modified}${connection}"
+        arm_id="${arm_id}"
+        arm_prefix="${arm_prefix_modified}"
+        ee_id="${ee_id}"
+        ee_inertials="${xacro.load_yaml('$(find franka_description)/end_effectors/$(arg ee_id)/inertials.yaml')}"
+        rpy_ee="$(arg rpy_ee)"
+        xyz_ee="$(arg xyz_ee)"
+        tcp_xyz="$(arg tcp_xyz)"
+        tcp_rpy="$(arg tcp_rpy)"
+        safety_distance="$(arg safety_distance)"
+        gazebo="${gazebo}"
+        description_pkg="$(arg description_pkg)"
+        with_sc="${with_sc}"
+      />
+    </xacro:if>
+    <!-- <xacro:if value="${hand and ee_id != 'none' and ee_id != 'franka_hand'}">
       <xacro:include filename="$(find franka_description)/end_effectors/common/ee_with_one_link.xacro"/>
       <xacro:include filename="$(find franka_description)/end_effectors/common/utils.xacro" />
@@ -90,5 +114,5 @@
         with_sc="${with_sc}"
       />
-    </xacro:if>
+    </xacro:if> -->
     <!-- Definition of additional Gazebo tags -->
     <xacro:if value="${gazebo}">
