Commit message: camera sim done, coordinate work needed

File: end_effectors/camera/camera_arguments.xacro (robot description, xacro)
@@ -6,7 +6,8 @@
   <xacro:arg name="ee_id" default="camera" />
   <!-- Position offset between ee and parent frame -->
-  <xacro:arg name="xyz_ee" default="0 0 0" />
+  <xacro:arg name="xyz_ee" default="0 0 0.05" />
   <!-- Rotation offset between ee and parent frame -->
-  <xacro:arg name="rpy_ee" default= "0 0 ${-pi/4}" />
+  <!-- <xacro:arg name="rpy_ee" default= "0 0 ${-pi/4}" /> -->
+  <xacro:arg name="rpy_ee" default= "0 ${0} ${-pi/4}" />
   <!-- Position offset between ee frame and tcp frame -->
   <xacro:arg name="tcp_xyz" default="0 0 0.1034" />

File: end_effectors/common/camera.xacro (robot description, xacro)
@@ -8,5 +8,5 @@
       <visual>
         <geometry>
-          <box size="0.05 0.05 0.05"/> <!-- 카메라 크기 -->
+          <box size="0.1 0.05 0.05"/> <!-- 카메라 크기 -->
         </geometry>
         <material name="camera_material">
@@ -16,5 +16,5 @@
       <collision>
         <geometry>
-          <box size="0.05 0.05 0.05"/>
+          <box size="0.1 0.05 0.05"/>
         </geometry>
       </collision>
@@ -47,11 +47,4 @@
             </clip>
           </camera>
-          <plugin
-            filename="libgazebo_ros_camera.so"
-            name="camera_controller">
-            <ros>
-              <namespace>/camera</namespace>
-            </ros>
-          </plugin>
         </sensor>
       </gazebo>
